File: badge00/badge00.sch (KiCad schematic (older format))
At the start: 11 parts, among them Q1 BC548, Q2 BC548

Commit message: upadate schematic
Parts:
- C1, C2: value 22uF -> 10uF
- R1, R4: value 150R -> 470R
Changed lines of the file:
@@
-EESchema Schematic File Version 2
+EESchema Schematic File Version 4
 LIBS:power
 LIBS:device
@@
 LIBS:valves
 LIBS:badge00-cache
-EELAYER 25 0
+EELAYER 26 0
 EELAYER END
 $Descr A4 11693 8268
@@
 P 5325 2750
 F 0 "R1" V 5405 2750 50  0000 C CNN
-F 1 "150R" V 5325 2750 50  0000 C CNN
+F 1 "470R" V 5325 2750 50  0000 C CNN
 F 2 "Resistors_THT:R_Axial_DIN0207_L6.3mm_D2.5mm_P10.16mm_Horizontal" V 5255 2750 50  0001 C CNN
 F 3 "" H 5325 2750 50  0001 C CNN
@@
 P 5600 3425
 F 0 "C1" H 5625 3525 50  0000 L CNN
-F 1 "22uF" H 5625 3325 50  0000 L CNN
+F 1 "10uF" H 5625 3325 50  0000 L CNN
 F 2 "Capacitors_THT:CP_Radial_D5.0mm_P2.50mm" H 5638 3275 50  0001 C CNN
 F 3 "" H 5600 3425 50  0001 C CNN
@@
 P 6550 2750
 F 0 "R4" V 6630 2750 50  0000 C CNN
-F 1 "150R" V 6550 2750 50  0000 C CNN
+F 1 "470R" V 6550 2750 50  0000 C CNN
 F 2 "Resistors_THT:R_Axial_DIN0207_L6.3mm_D2.5mm_P10.16mm_Horizontal" V 6480 2750 50  0001 C CNN
 F 3 "" H 6550 2750 50  0001 C CNN
@@
 P 6300 3400
 F 0 "C2" H 6325 3500 50  0000 L CNN
-F 1 "22uF" H 6325 3300 50  0000 L CNN
+F 1 "10uF" H 6325 3300 50  0000 L CNN
 F 2 "Capacitors_THT:CP_Radial_D5.0mm_P2.50mm" H 6338 3250 50  0001 C CNN
 F 3 "" H 6300 3400 50  0001 C CNN
@@
 $EndComp
 Wire Wire Line
-	5325 3275 5325 3500
+	5325 3275 5325 3425
 Wire Wire Line
 	5450 3425 5325 3425
 Connection ~ 5325 3425
 Wire Wire Line
-	6550 3300 6550 3500
+	6550 3300 6550 3400
 Wire Wire Line
 	6450 3400 6550 3400
@@
 	5325 2900 5325 2975
 Wire Wire Line
-	5825 2900 5825 3600
+	5825 2900 5825 3425
 Wire Wire Line
 	5825 3425 5750 3425
@@
 	6100 2900 6100 3400
 Wire Wire Line
-	6000 3400 6150 3400
+	6000 3400 6100 3400
 Wire Wire Line
 	6550 2450 6550 2600
 Wire Wire Line
-	4675 2450 6550 2450
+	4675 2450 5325 2450
 Wire Wire Line
 	5325 2450 5325 2600
@@
 	5325 3900 5325 4025
 Wire Wire Line
-	4675 4025 6550 4025
+	4675 4025 5325 4025
 Wire Wire Line
 	6550 4025 6550 3900
@@
 	4675 4025 4675 3425
 Connection ~ 5325 4025
+Wire Wire Line
+	5325 3425 5325 3500
+Wire Wire Line
+	6550 3400 6550 3500
+Wire Wire Line
+	5825 2450 6100 2450
+Wire Wire Line
+	6100 2450 6550 2450
+Wire Wire Line
+	6100 3400 6150 3400
+Wire Wire Line
+	5825 3425 5825 3600
+Wire Wire Line
+	5325 2450 5825 2450
+Wire Wire Line
+	5325 4025 6550 4025
 $EndSCHEMATC
