File: badge00/badge00.sch (KiCad schematic (older format))
At the start: 11 parts, among them Q1 BC548, Q2 BC548

Commit message: re-layout
Parts:
- Q1, Q2: footprint TO_SOT_Packages_THT:TO-92_Inline_Narrow_Oval -> library:TO-92_Inline_Wide
Changed lines of the file:
@@
 F 0 "Q1" H 5625 3775 50  0000 L CNN
 F 1 "BC548" H 5625 3700 50  0000 L CNN
-F 2 "TO_SOT_Packages_THT:TO-92_Inline_Narrow_Oval" H 5625 3625 50  0001 L CIN
+F 2 "library:TO-92_Inline_Wide" H 5625 3625 50  0001 L CIN
 F 3 "" H 5425 3700 50  0001 L CNN
 	1    5425 3700
@@
 F 0 "Q2" H 6650 3775 50  0000 L CNN
 F 1 "BC548" H 6650 3700 50  0000 L CNN
-F 2 "TO_SOT_Packages_THT:TO-92_Inline_Narrow_Oval" H 6650 3625 50  0001 L CIN
+F 2 "library:TO-92_Inline_Wide" H 6650 3625 50  0001 L CIN
 F 3 "" H 6450 3700 50  0001 L CNN
 	1    6450 3700

Commit message: switch
Parts:
- added SW1: SW_SPDT, library:SW_HH_SS12D07-G4-2, symbol Switch:SW_SPDT
Connections:
- wire segments 33 -> 34
Changed lines of the file:
@@
 	5325 3900 5325 4025
-Wire Wire Line
-	4675 4025 5325 4025
 Wire Wire Line
 	6550 4025 6550 3900
@@
 	4675 2450 4675 3125
 Connection ~ 5325 2450
-Wire Wire Line
-	4675 4025 4675 3425
 Connection ~ 5325 4025
 Wire Wire Line
@@
 Wire Wire Line
 	5325 4025 6550 4025
+$Comp
+L Switch:SW_SPDT SW1
+U 1 1 5BA56C60
+P 4775 3700
+F 0 "SW1" V 4821 3512 50  0000 R CNN
+F 1 "SW_SPDT" V 4730 3512 50  0000 R CNN
+F 2 "library:SW_HH_SS12D07-G4-2" H 4775 3700 50  0001 C CNN
+F 3 "" H 4775 3700 50  0001 C CNN
+	1    4775 3700
+	0    -1   -1   0
+$EndComp
+Wire Wire Line
+	4675 3425 4675 3500
+Wire Wire Line
+	4775 3900 4775 4025
+Wire Wire Line
+	4775 4025 5325 4025
 $EndSCHEMATC

Commit message: bom
Parts:
- SW1: value SW_SPDT -> SS12D07
Changed lines of the file:
@@
 P 4775 3700
 F 0 "SW1" V 4821 3512 50  0000 R CNN
-F 1 "SW_SPDT" V 4730 3512 50  0000 R CNN
+F 1 "SS12D07" V 4775 4125 50  0000 R CNN
 F 2 "library:SW_HH_SS12D07-G4-2" H 4775 3700 50  0001 C CNN
 F 3 "" H 4775 3700 50  0001 C CNN
