File: badge00/badge00.kicad_pcb (KiCad board)
At the start: 2 copper layers, 40 x 40 mm, 15 parts, among them Q1 BC548, Q2 BC548

Commit message: re-layout
Parts:
- removed the G*** at (128.0, 68.0)
- added G***: LOGO, Graphics:robot2_35x35, F.Cu at (128.1, 67.9)
- added G***: LOGO, Graphics:logo-franzininho12_7, F.Cu at (117.1, 79.8)
- C1, C2: value 22uF -> 10uF
- Q1, Q2: footprint TO_SOT_Packages_THT:TO-92_Inline_Narrow_Oval -> library:TO-92_Inline_Wide
- R1, R4: value 150R -> 470R
- moved Q1 1.80 mm to (125.1, 52.7)
- moved Q2 0.57 mm to (139.7, 52.7)
- moved G*** 0.25 mm to (144.5, 51.7)
- moved G*** 0.07 mm to (144.5, 52.1)
Routing:
- net Net-(BT1-Pad2): track 49.5 -> 0.00 mm, vias 1 -> 0
- net Net-(C2-Pad2): track 56.5 -> 61.2 mm
- net Net-(C1-Pad2): track 57.9 -> 60.0 mm
- net Net-(C1-Pad1): track 28.4 -> 26.9 mm
Other:
- board text added: "+"
- board text added: "V0RV1"
- board text removed: "V0RV0"

Commit message: switch
Parts:
- removed the G*** at (144.5, 51.7)
- removed the G*** at (144.5, 52.1)
- added REF***: OSHW-Logo_7.5x8mm_SilkScreen, Symbols:OSHW-Logo_7.5x8mm_SilkScreen, B.Cu at (145.0, 51.8)
- added REF***: KiCad-Logo2_6mm_SilkScreen, Symbols:KiCad-Logo2_6mm_SilkScreen, B.Cu at (142.5, 82.8)
- added SW1: SW_SPDT, library:SW_HH_SS12D07-G4-2, B.Cu at (114.3, 81.8)
- moved G*** 38.3 mm to (144.3, 52.8)
Connections:
- Q1 pad 3: Net-(BT1-Pad2) -> Net-(Q1-Pad3)
- Q2 pad 3: Net-(BT1-Pad2) -> Net-(Q1-Pad3)
Routing:
- net Net-(BT1-Pad2): track 0.00 -> 23.1 mm
- added copper zone on B.Cu, net Net-(Q1-Pad3)
- added copper zone on F.Cu, net Net-(Q1-Pad3)
- removed copper zone on B.Cu, net Net-(BT1-Pad2)
- removed copper zone on F.Cu, net Net-(BT1-Pad2)
Other:
- board text removed: "10^-3 = m - mili 10^-6 = u - micro 10^-9 = n - nano 10^-12= p - pico"
- board text removed: "10^3 = k - kilo 10^6 = M - mega 10^9 = G - giga 10^12 = T - tera"
- board text removed: "Lei de Ohm"
- board text removed: "V = R x I"
